Commit message: feat: prepare dev-v4 manipulation runtime

File: src/bringup/marvin_manipulation/rt_launch/urdf/marvin_manipulation.urdf.xacro (robot description, xacro)
@@ -9,6 +9,5 @@
      Args: same stand/arm mounts as marvin.urdf.xacro, plus
        left_gripper_serial_port / right_gripper_serial_port /
-       with_gripper (master; false = grippers not installed) /
-       with_left_gripper / with_right_gripper (per side)
+       load_pika_hardware (true = both grippers; false = neither)
      Actuated: left_/right_gripper_left_joint (right finger URDF-mimic). -->
 <robot xmlns:xacro="http://www.ros.org/wiki/xacro" name="marvin_manipulation">
@@ -32,7 +31,5 @@
   <xacro:arg name="left_gripper_serial_port" default="/dev/pika_left_gripper"/>
   <xacro:arg name="right_gripper_serial_port" default="/dev/pika_right_gripper"/>
-  <xacro:arg name="with_gripper" default="true"/>
-  <xacro:arg name="with_left_gripper" default="true"/>
-  <xacro:arg name="with_right_gripper" default="true"/>
+  <xacro:arg name="load_pika_hardware" default="true"/>
   <!-- Pika TCP + finger limits owned by this bringup (edit config/model/*.yaml). -->
   <xacro:arg name="gripper_tcp_file"
@@ -55,6 +52,5 @@
     right_base_xyz="$(arg right_base_xyz)"
     right_base_rpy="$(arg right_base_rpy)"/>
-  <xacro:if value="$(arg with_gripper)">
-    <xacro:if value="$(arg with_left_gripper)">
+  <xacro:if value="$(arg load_pika_hardware)">
       <xacro:marvin_pika_adaptor prefix="left_" parent="flange_L"/>
       <xacro:pika_gripper
@@ -63,8 +59,6 @@
         tcp_file="$(arg gripper_tcp_file)"
         joint_limits_file="$(arg gripper_joint_limits_file)">
-        <origin xyz="0 0 0.004" rpy="0 0 ${3*pi/4}"/>
+        <origin xyz="0 0 0.004" rpy="0 0 ${-3*pi/4}"/>
       </xacro:pika_gripper>
-    </xacro:if>
-    <xacro:if value="$(arg with_right_gripper)">
       <xacro:marvin_pika_adaptor prefix="right_" parent="flange_R"/>
       <xacro:pika_gripper
@@ -73,7 +67,6 @@
         tcp_file="$(arg gripper_tcp_file)"
         joint_limits_file="$(arg gripper_joint_limits_file)">
-        <origin xyz="0 0 0.004" rpy="0 0 ${pi/4}"/>
+        <origin xyz="0 0 0.004" rpy="0 0 ${-pi/4}"/>
       </xacro:pika_gripper>
-    </xacro:if>
   </xacro:if>
   <xacro:if value="$(arg ros2_control)">
@@ -85,6 +78,5 @@
       stale_error_ms="$(arg stale_error_ms)"
       max_joint_velocity="$(arg max_joint_velocity)"/>
-    <xacro:if value="$(arg with_gripper)">
-      <xacro:if value="$(arg with_left_gripper)">
+    <xacro:if value="$(arg load_pika_hardware)">
         <xacro:pika_gripper_ros2_control
           name="LeftPikaGripperHardware"
@@ -93,6 +85,4 @@
           joint_limits_file="$(arg gripper_joint_limits_file)"
           use_fake_hardware="$(arg use_fake_hardware)"/>
-      </xacro:if>
-      <xacro:if value="$(arg with_right_gripper)">
         <xacro:pika_gripper_ros2_control
           name="RightPikaGripperHardware"
@@ -101,5 +91,4 @@
           joint_limits_file="$(arg gripper_joint_limits_file)"
           use_fake_hardware="$(arg use_fake_hardware)"/>
-      </xacro:if>
     </xacro:if>
   </xacro:if>
